Commit message: fix: Fix the gears pushing themselves
-  Change selfCollide to false for the gripper components
- Add a collision filter to prevent the gripper parts from interacting with each other

File: urdf/arm_assem_urdf_v3.urdf (robot description, URDF)
Before this commit: robot arm_assem_urdf_v3, 12 links, 11 joints
Links:
- removed link l_elbo
- removed link r_elbo
Joints:
- removed joint l_j_elbo
- removed joint r_j_elbo
- joint Lgripperjoint: mimic (none) -> joint=rgripper_joint multiplier=1.0 offset=0.0
- joint l_fing_j: mimic (none) -> joint=r_fingerj multiplier=1.0 offset=0.0
