Commit message: feat: Enhance gripper control and update configurations for Lgripperjoint, Update the poses to be more real

File: arm_assem_urdf_v3/urdf/arm_assem_urdf_v3.urdf (robot description, URDF)
Before this commit: robot arm_assem_urdf_v3, 11 links, 10 joints
Joints:
- joint Lgripperjoint: mimic joint=rgripper_joint multiplier=1.0 offset=0.0 -> (none)
- joint l_fing_j: mimic joint=r_fingerj multiplier=1.0 offset=0.0 -> (none)

File: move/config/gazebo_arm_assem_urdf_v3.urdf (robot description, URDF)
Before this commit: robot arm_assem_urdf_v3, 11 links, 10 joints
Joints:
- joint Lgripperjoint: mimic joint=rgripper_joint multiplier=1.0 offset=0.0 -> (none)
- joint rgripper_joint: mimic (none) -> joint=Lgripperjoint multiplier=1.0 offset=0.0
